Commit message: fix: put the sensor where it actually is, 0.725 m up
The mount height was 0.30 m in five files and in both sensor joints of the
hardware URDF. It was never measured - it was a placeholder that everything
else got anchored to, including the URDF, whose x and y ARE measured (the
0727 spin fit: 0.517 m forward, 0.173 m left of the axle) and whose z was
back-derived from the placeholder.

Tape says 0.725 m to the Livox optical origin. The 0727 map agrees to
within 0.05 m and rules out 0.30 m outright: sampling the merged cloud
under the recorded trajectory, restricted to patches whose ground is flat
to 0.10 m so a kerb alongside cannot masquerade as the surface, puts the
sensor 0.775 m up with sd 0.018 - and three sampling radii from 0.3 to
0.8 m agree to 8 mm. The 0.05 m gap is most likely the optical origin
sitting inside the housing above whatever the tape reached. 0.725 is the
conservative of the two here: understating the mount can only make the
guard less eager, where overstating it reads the ground as an obstacle.

This was not cosmetic. Obstacle height is `z + sensor_height`, so a mount
understated by 0.425 m slid the entire detection band up with it. The
gate's nominal 0.15-1.9 m window was really watching 0.575-2.325 m above
ground: a bollard, a kerb, a suitcase, a crouching child - anything under
57 cm - did not exist as far as the chair was concerned. It now sees from
15 cm, which is also why obstacle stops should be expected to fire more
often than they used to.

Two things follow from the correction and are fixed with it. The rider
exclusion box in obstacle_clusters is in raw lidar z, so its -0.5 floor
went from 0.2 m below the ground plane to 0.225 m above it, leaving the
rider's feet and the footrest outside the box - and an obstacle that
travels with the chair is exactly what the new tracker would confirm as
parked. It is now tied to SENSOR_HEIGHT_M. And the follower's ground-blind
radius, quoted as 2.4 m, is 0.725/tan(7 deg) = 5.9 m; the safety band has
been carrying more of the drop safety than the docstring admitted.

test_mount_geometry pins all of it together - the three consumers, the
follower default, both URDF joints through the built-in extrinsic, the
exclusion floor, and the docstring radius - because one number living in
six files is what produced this.

File: src/wheelchair_description/urdf/wheelchair_hardware.urdf.xacro (robot description, xacro)
@@ -15,4 +15,12 @@
   Re-measure it whenever the sensor mount moves. The remaining legacy chassis
   dimensions are copied, not newly certified physical measurements.
+  Sensor height is measured, as of 2026-07-31: the Livox optical origin sits
+  0.725 m above the ground, and imu_link follows from it through the built-in
+  extrinsic (0.725 - 0.04412). It was 0.300 m here, which was never a
+  measurement - it was the placeholder SENSOR_HEIGHT_M the perception code
+  carried, and both the lidar and the IMU height were anchored to it. The
+  0727 map disagrees with it by 0.47 m: sampling the merged cloud under 77
+  flat patches of the recorded trajectory puts the lidar 0.775 m up
+  (sd 0.018), which is 0.05 m above the tape and nowhere near 0.300.
 -->
 <robot name="wheelchair_hardware" xmlns:xacro="http://www.ros.org/wiki/xacro">
@@ -174,5 +182,5 @@
     <parent link="base_link"/>
     <child link="lidar_link"/>
-    <origin xyz="0.246 0.14971 0.300" rpy="0 0 0"/>
+    <origin xyz="0.246 0.14971 0.725" rpy="0 0 0"/>
   </joint>
   <link name="imu_link"/>
@@ -180,5 +188,5 @@
     <parent link="base_link"/>
     <child link="imu_link"/>
-    <origin xyz="0.257 0.173 0.25588" rpy="0 0 0"/>
+    <origin xyz="0.257 0.173 0.68088" rpy="0 0 0"/>
   </joint>
   <link name="body"/>

Commit message: feat: drive the 0727 line about the point it was recorded about
The mount offset is now the operator's measurement, 0.500 m forward and
0.200 m left of the axle, superseding the 0.517/0.173 fitted from six
in-place rotations. The two agree to within that fit's own +-0.03 m
between-spin spread, so this is a sharper instrument rather than a
contradiction: a tape reaches the axle directly, where the fit had to infer
it from how the chair turned. Both URDF sensor joints follow, imu_link
directly and lidar_link through the built-in extrinsic.

That leaves the 0727 route, which was built about the old offset and says
so in chair_centre_in_body_xyz. The follower was ignoring that field and
correcting poses with whatever the constant happened to be, so changing the
constant would have slid the entire recorded path 0.032 m sideways while
still reporting it as tracking. It now drives a route about the point the
route was recorded about, and warns when that differs from the current
measurement - because it does differ, and what it costs is that the band's
clearances are stated about a point 0.032 m from where the chair centre
actually is. Reproducing the drive and knowing where the wheels are are two
different questions and the route only answers the first.

Nothing is shifted or regenerated. Route and pose share a reference point,
so the chair reproduces the recorded line exactly, which is the property
today's run depends on.

trial_0727.sh / go.sh / stop.sh are what gets typed at the chair. The trial
brings the stack up with the discretionary guards off - the run measures
whether localization stays attached over 383 m, and a band refusal or a
geofence trip would end that measurement while looking, from outside, like
exactly what it was meant to detect. Cluster avoidance stays on, because it
is not behind that switch. go refuses rather than starts if the follower is
absent, the object tracker is silent, or localization is not TRACKING, and
it checks all three before commanding anything - a check after the first
command runs while the chair is already moving. stop checks nothing, since
a stop that refuses on a failed precondition is not a stop.

All three install alongside the bringup with the same checksum verification:
they live in $HOME, outside the checkout, which is how the bringup was once
found still launching the previous week's route.

File: src/wheelchair_description/urdf/wheelchair_hardware.urdf.xacro (robot description, xacro)
@@ -12,7 +12,12 @@
     imu_link/body   FAST-LIO built-in IMU body origin
     lidar_link      Livox optical origin
-  The horizontal body offset was fitted from six physical in-place rotations.
-  Re-measure it whenever the sensor mount moves. The remaining legacy chassis
-  dimensions are copied, not newly certified physical measurements.
+  The horizontal body offset is measured: imu_link sits 0.500 m forward and
+  0.200 m left of the axle midpoint (operator, 2026-07-31). It supersedes the
+  0.517/0.173 fitted from six in-place rotations, which it agrees with to
+  within that fit's own +-0.03 m spread. Routes recorded under the fitted
+  value still carry it and are still driven about it - see
+  body_frame.route_chair_centre. Re-measure whenever the mount moves; nothing
+  detects that on its own. The remaining legacy chassis dimensions are copied,
+  not newly certified physical measurements.
   Sensor height is measured, as of 2026-07-31: the Livox optical origin sits
   0.725 m above the ground, and imu_link follows from it through the built-in
@@ -182,5 +187,5 @@
     <parent link="base_link"/>
     <child link="lidar_link"/>
-    <origin xyz="0.246 0.14971 0.725" rpy="0 0 0"/>
+    <origin xyz="0.229 0.17671 0.725" rpy="0 0 0"/>
   </joint>
   <link name="imu_link"/>
@@ -188,5 +193,5 @@
     <parent link="base_link"/>
     <child link="imu_link"/>
-    <origin xyz="0.257 0.173 0.68088" rpy="0 0 0"/>
+    <origin xyz="0.240 0.200 0.68088" rpy="0 0 0"/>
   </joint>
   <link name="body"/>
